File: Phase_B_ATMEGA_v3/Phase_B_ATMEGA_v3.kicad_pcb (KiCad board)
At the start: 2 copper layers, 49 parts, among them J1 AVR-ISP-6, J2 USB_B_Mini, J3 ESP_Conn, U1 CA56-12EWA, U2 74HC595, U3 ATmega32U4-A, U4 USBLC6-2SC6, U5 LP2985-3.3, Y1 16MHz

Commit message: 1
Parts:
- moved S1 68.0 mm to (120.7, 130.8)
- moved S3 66.5 mm to (171.4, 62.2)
- moved C8 65.6 mm to (112.6, 113.3), turned to 90 degrees
- moved R12 64.8 mm to (113.0, 79.7), turned to 90 degrees
- moved C4 62.7 mm to (116.6, 113.8), turned to 90 degrees
- moved C10 62.2 mm to (126.6, 113.8), turned to 90 degrees
- moved R11 60.2 mm to (116.8, 79.7), turned to 90 degrees
- moved C5 59.1 mm to (119.1, 113.8), turned to 90 degrees
- moved C11 58.7 mm to (129.2, 113.8), turned to 90 degrees
- moved C13 57.2 mm to (111.6, 90.2)
- moved C14 57.2 mm to (111.6, 92.7)
- moved D1 56.9 mm to (113.0, 109.2)
- moved R10 55.7 mm to (120.7, 79.7), turned to 90 degrees
- moved C6 55.6 mm to (121.6, 113.8), turned to 90 degrees
- moved D2 54.4 mm to (113.0, 106.7)
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Other:
- board outline added: 78.7 x 99.1 mm
- board text added: "DU Embedded Systems ENCE 3231 Phase B Kitchen Timer"
- board text added: "Daniel Silva Rios"
- board text added: "Increment"
- board text added: "Start/Stop"

Commit message: 1
Parts:
- J1: moved to B.Cu
- moved D1 45.5 mm to (110.5, 63.8), turned to -90 degrees
- moved D2 42.8 mm to (113.0, 63.8), turned to -90 degrees
- moved R3 41.3 mm to (110.5, 68.6), turned to 90 degrees
- moved R4 38.4 mm to (113.0, 68.6), turned to 90 degrees
- moved C8 38.1 mm to (146.1, 94.9)
- moved R16 36.9 mm to (164.2, 95.2)
- moved R13 36.4 mm to (149.2, 95.9), turned to 0 degrees
- moved S3 35.8 mm to (154.9, 94.0)
- moved D3 35.8 mm to (160.8, 95.0)
- moved C6 32.2 mm to (152.6, 105.3), turned to 0 degrees
- moved C5 31.2 mm to (144.1, 95.1)
- moved C7 28.8 mm to (152.7, 110.0), turned to 0 degrees
- moved J2 27.3 mm to (179.1, 108.0), turned to 90 degrees
- moved C10 20.8 mm to (147.3, 116.0), turned to -90 degrees
- moved C4 19.7 mm to (133.2, 103.2), turned to 180 degrees
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Routing:
- net +5V: track 0.00 -> 228.7 mm, vias 0 -> 2
- net Dig1: track 0.00 -> 80.1 mm, vias 0 -> 4
- net Buzzer: track 0.00 -> 62.4 mm, vias 0 -> 2
- net RED_LED: track 0.00 -> 60.0 mm, vias 0 -> 2
- net SH_CP: track 0.00 -> 58.7 mm
- net Dig4: track 0.00 -> 58.4 mm, vias 0 -> 2
- net Dig3: track 0.00 -> 57.5 mm, vias 0 -> 2
- net GND: track 0.00 -> 56.1 mm, vias 0 -> 35
- net GREEN_LED: track 0.00 -> 54.6 mm, vias 0 -> 2
- net Dig2: track 0.00 -> 54.5 mm, vias 0 -> 2
- net Button_1: track 0.00 -> 41.6 mm, vias 0 -> 2
- net Button_2: track 0.00 -> 40.8 mm, vias 0 -> 2
- net Net-(U1-b): track 0.00 -> 33.3 mm, vias 0 -> 2
- net +3.3V: track 0.00 -> 33.0 mm
- net TX: track 0.00 -> 31.0 mm, vias 0 -> 2
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- added copper zone on B.Cu, net GND
